File: Hardware/Peripheral/mkrd-002.brd (EAGLE design)
At the start: 25 x 26 mm, 5 parts, among them J1 MKR

Commit message: Added new board.
Other:
- board text added: "MKR Display II 0.0.1-X"
- board text removed: "MKR Display 0.0.1-X"
Changed lines of the file:
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@@
 <layer number="20" name="Dimension" color="24" fill="1" visible="yes" active="yes"/>
 <layer number="21" name="tPlace" color="7" fill="1" visible="yes" active="yes"/>
-<layer number="22" name="bPlace" color="7" fill="1" visible="no" active="yes"/>
+<layer number="22" name="bPlace" color="7" fill="1" visible="yes" active="yes"/>
 <layer number="23" name="tOrigins" color="15" fill="1" visible="yes" active="yes"/>
 <layer number="24" name="bOrigins" color="15" fill="1" visible="yes" active="yes"/>
 <layer number="25" name="tNames" color="7" fill="1" visible="yes" active="yes"/>
-<layer number="26" name="bNames" color="7" fill="1" visible="no" active="yes"/>
+<layer number="26" name="bNames" color="7" fill="1" visible="yes" active="yes"/>
 <layer number="27" name="tValues" color="7" fill="1" visible="no" active="yes"/>
 <layer number="28" name="bValues" color="7" fill="1" visible="no" active="yes"/>
@@
 <rectangle x1="24" y1="0" x2="25" y2="26" layer="41"/>
 <rectangle x1="0" y1="0" x2="7.5" y2="1" layer="41"/>
-<text x="12.5" y="15.5" size="1" layer="26" rot="MR0" align="center">MKR Display 0.0.1-X</text>
+<text x="12.5" y="15.5" size="1" layer="26" rot="MR0" align="center">MKR Display II 0.0.1-X</text>
 <hole x="23" y="2" drill="2"/>
 <hole x="23" y="24" drill="2"/>
