File: Hardware/Peripheral/mkrd-001.brd (EAGLE design)
At the start: 32 x 32 mm, 11 parts, among them J1 MKR, X1 AQM0802A-RN-GBW

Commit message: Signal name.
Connections:
- net N$1 renamed LCDVOUT
- net N$2 renamed CAP1P
- net N$3 renamed CAP1N
Changed lines of the file:
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@@
 <wire x1="19.9644" y1="26.0604" x2="20" y2="26" width="0.1524" layer="1"/>
 </signal>
-<signal name="N$2">
+<signal name="CAP1P">
 <contactref element="X1" pad="4"/>
 <contactref element="C3" pad="2"/>
@@
 <wire x1="26.2128" y1="2.1336" x2="26.27" y2="2" width="0.1524" layer="16"/>
 </signal>
-<signal name="N$3">
+<signal name="CAP1N">
 <contactref element="C3" pad="1"/>
 <contactref element="X1" pad="3"/>
@@
 <wire x1="23.622" y1="2.1336" x2="23.73" y2="2" width="0.1524" layer="1"/>
 </signal>
-<signal name="N$1">
+<signal name="LCDVOUT">
 <contactref element="X1" pad="2"/>
 <contactref element="C2" pad="2"/>
