File: Hardware/Peripheral/mkrd-001.brd (EAGLE design)
At the start: 32 x 32 mm, 11 parts, among them J1 MKR, X1 AQM0802A-RN-GBW

Commit message: Silk.
Parts:
- renumbered X1 to LCD1
Other:
- board text added: "103"
- board text added: "104"
- board text added: "152"
- board text added: "1u"
- board text added: "332"
Changed lines of the file:
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@@
 <setting verticaltext="up"/>
 </settings>
-<grid distance="1" unitdist="mm" unit="mm" style="lines" multiple="1" display="yes" altdistance="5" altunitdist="mil" altunit="mil"/>
+<grid distance="0.5" unitdist="mm" unit="mm" style="lines" multiple="2" display="yes" altdistance="5" altunitdist="mil" altunit="mil"/>
 <layers>
 <layer number="1" name="Top" color="4" fill="1" visible="yes" active="yes"/>
@@
 <rectangle x1="10" y1="9.5" x2="22" y2="14.5" layer="42"/>
 <text x="16" y="31" size="1" layer="26" rot="MR0" align="center">MKR</text>
+<text x="19" y="2" size="1" layer="25" rot="R90" align="center">104</text>
+<text x="10" y="2" size="1" layer="25" rot="R90" align="center">1u</text>
+<text x="28" y="2" size="1" layer="25" rot="R90" align="center">1u</text>
+<text x="6" y="27.5" size="1" layer="25" rot="R90" align="center">152</text>
+<text x="8.5" y="27.5" size="1" layer="25" rot="R90" align="center">332</text>
+<text x="23.5" y="27.5" size="1" layer="25" rot="R90" align="center">103</text>
+<text x="26" y="27.5" size="1" layer="25" rot="R90" align="center">103</text>
 </plain>
 <attributes>
@@
 <attribute name="VALUE" x="17.778" y="4.667" size="1.27" layer="27" ratio="10" rot="R180"/>
 </element>
-<element name="X1" library="AQM0802A-RN-GBW" package="AQM0802A-RN-GBW-FOOTPRINT" value="AQM0802A-RN-GBW" x="16" y="4" smashed="yes">
+<element name="LCD1" library="AQM0802A-RN-GBW" package="AQM0802A-RN-GBW-FOOTPRINT" value="AQM0802A-RN-GBW" x="16" y="4" smashed="yes">
 <attribute name="NAME" x="16" y="6" size="1" layer="25" align="center"/>
 <attribute name="VALUE" x="16" y="2" size="1" layer="27" align="center"/>
@@
 <contactref element="C1" pad="2"/>
 <contactref element="R2" pad="1"/>
-<contactref element="X1" pad="6"/>
+<contactref element="LCD1" pad="6"/>
 <wire x1="10.9728" y1="24.9936" x2="8.5344" y2="24.9936" width="0.1524" layer="1"/>
 <wire x1="11.8872" y1="25.908" x2="10.9728" y2="24.9936" width="0.1524" layer="1"/>
@@
 <contactref element="J1" pad="3"/>
 <contactref element="R3" pad="2"/>
-<contactref element="X1" pad="8"/>
+<contactref element="LCD1" pad="8"/>
 <wire x1="20.4216" y1="21.4884" x2="20.4216" y2="4.1148" width="0.1524" layer="1"/>
 <wire x1="16.002" y1="25.908" x2="20.4216" y2="21.4884" width="0.1524" layer="1"/>
@@
 <contactref element="J1" pad="2"/>
 <contactref element="R4" pad="2"/>
-<contactref element="X1" pad="7"/>
+<contactref element="LCD1" pad="7"/>
 <wire x1="18.8976" y1="21.0312" x2="18.8976" y2="4.1148" width="0.1524" layer="1"/>
 <wire x1="14.0208" y1="25.908" x2="18.8976" y2="21.0312" width="0.1524" layer="1"/>
@@
 <contactref element="R3" pad="1"/>
 <contactref element="R4" pad="1"/>
-<contactref element="X1" pad="9"/>
+<contactref element="LCD1" pad="9"/>
 <contactref element="C1" pad="1"/>
-<contactref element="X1" pad="5"/>
+<contactref element="LCD1" pad="5"/>
 <contactref element="C2" pad="1"/>
 <wire x1="15.0876" y1="4.8768" x2="15.8496" y2="4.1148" width="0.1524" layer="1"/>
@@
 </signal>
 <signal name="CAP1P">
-<contactref element="X1" pad="4"/>
+<contactref element="LCD1" pad="4"/>
 <contactref element="C3" pad="2"/>
 <wire x1="15.6972" y1="2.8956" x2="14.6304" y2="3.9624" width="0.1524" layer="16"/>
@@
 <signal name="CAP1N">
 <contactref element="C3" pad="1"/>
-<contactref element="X1" pad="3"/>
+<contactref element="LCD1" pad="3"/>
 <wire x1="14.1732" y1="2.8956" x2="13.1064" y2="3.9624" width="0.1524" layer="1"/>
 <wire x1="22.86" y1="2.8956" x2="14.1732" y2="2.8956" width="0.1524" layer="1"/>
@@
 </signal>
 <signal name="LCDVOUT">
-<contactref element="X1" pad="2"/>
+<contactref element="LCD1" pad="2"/>
 <contactref element="C2" pad="2"/>
 <wire x1="9.6012" y1="2.1336" x2="11.43" y2="3.9624" width="0.1524" layer="1"/>
